Commit message: updated urdf

File: ros_basics_exercise/urdf/thymio_simple.urdf (robot description, URDF)
Before this commit: robot thymio, 3 links, 2 joints
Joints:
- joint left_wheel_joint: origin xyz=-0.03 0.056 -0.0100 rpy=0 0 0 -> xyz=-0.03 0.056 -0.0100 rpy=1.57079632679 0 0
- joint right_wheel_joint: origin xyz=-0.03 -0.056 -0.0100 rpy=0 0 0 -> xyz=-0.03 -0.056 -0.0100 rpy=1.57079632679 0 0

File: ros_basics_exercise/urdf/thymio_simple.urdf.xacro (robot description, xacro)
@@ -30,19 +30,4 @@
             <material name="white"/>
         </collision>
-        <!-- Implement the caster wheel -->
-        <visual>
-            <origin xyz="0.03 0 -0.0225" rpy="0 0 0"/>
-            <geometry>
-                <sphere radius="0.0095"/>
-            </geometry>
-            <material name="white"/>
-        </visual>
-        <collision>
-            <origin xyz="0.03 0 -0.0225" rpy="0 0 0"/>
-            <geometry>
-                <sphere radius="0.0095"/>
-            </geometry>
-            <material name="white"/>
-        </collision>
         <inertial>
 			<mass value="${body_mass}"/>
@@ -50,8 +35,25 @@
 		</inertial>
     </link>
+    <!-- Implement the caster wheel -->
+    <link name="caster_wheel">
+		<visual>
+		    <origin xyz="0 0 0" rpy="0 0 0"/>
+		    <geometry>
+		        <sphere radius="0.0095"/>
+		    </geometry>
+		    <material name="white"/>
+		</visual>
+		<collision>
+		    <origin xyz="0 0 0" rpy="0 0 0"/>
+		    <geometry>
+		        <sphere radius="0.0095"/>
+		    </geometry>
+		    <material name="white"/>
+		</collision>
+	</link>
     <!-- Implement the left wheel -->
     <link name="left_wheel">
         <visual>
-            <origin xyz="0 0 0" rpy="1.57079632679 0 0"/>
+            <origin xyz="0 0 0" rpy="${pi/2} 0 0"/>
             <geometry>
                 <cylinder length="${wheel_len}" radius="${wheel_radius}"/>
@@ -60,5 +62,5 @@
         </visual>
         <collision>
-           <origin xyz="0 0 0" rpy="1.57079632679 0 0"/>
+           <origin xyz="0 0 0" rpy="${pi/2} 0 0"/>
             <geometry>
                 <cylinder length="${wheel_len}" radius="${wheel_radius}"/>
@@ -74,5 +76,5 @@
     <link name="right_wheel">
         <visual>
-            <origin xyz="0 0 0" rpy="1.57079632679 0 0"/>
+            <origin xyz="0 0 0" rpy="${pi/2} 0 0"/>
             <geometry>
                 <cylinder length="${wheel_len}" radius="${wheel_radius}"/>
@@ -81,5 +83,5 @@
         </visual>
         <collision>
-           <origin xyz="0 0 0" rpy="1.57079632679 0 0"/>
+           <origin xyz="0 0 0" rpy="${pi/2} 0 0"/>
             <geometry>
                 <cylinder length="${wheel_len}" radius="${wheel_radius}"/>
@@ -92,10 +94,17 @@
 		</inertial>
     </link>
+    <!-- Implement the joint for the caster wheel -->
+	<joint name="caster_wheel_joint" type="fixed">
+		<parent link="base_link"/>
+		<child link="caster_wheel"/>
+		<origin xyz="0.03 0 -0.0225" rpy="0 0 0"/>
+		<axis xyz="0 0 0"/>
+	</joint>
     <!-- Implement the joint for the left wheel -->
 	<joint name="left_wheel_joint" type="continuous">
 		<parent link="base_link"/>
 		<child link="left_wheel"/>
-		<axis rpy="0 0 0" xyz="0 1 0"/>
 		<origin xyz="-0.03 0.056 -0.0100" rpy="0 0 0"/>
+		<axis xyz="0 1 0"/>
 	</joint>
     <!-- Implement the joint for the right wheel -->
@@ -103,6 +112,6 @@
 		<parent link="base_link"/>
 		<child link="right_wheel"/>
-		<axis rpy="0 0 0" xyz="0 1 0"/>
 		<origin xyz="-0.03 -0.056 -0.0100" rpy="0 0 0"/>
+		<axis xyz="0 1 0"/>
 	</joint>
     <!-- Add your sensors using the macro -->
