Commit message: urdf update

File: ros_basics_exercise/urdf/thymio_simple.urdf.xacro (robot description, xacro)
@@ -13,6 +13,7 @@
     <xacro:arg name="mass" default="0.270"/>
     <xacro:property name="mass_p" value="$(arg mass)"/>
-    <xacro:property name="body_mass" value="${mass_p * 0.80}"/>
+    <xacro:property name="body_mass" value="${mass_p * 0.75}"/>
     <xacro:property name="wheel_mass" value="${mass_p * 0.10}"/>
+    <xacro:property name="caster_mass" value="${mass_p * 0.05}"/>
     <link name="base_link">
         <visual>
@@ -51,4 +52,8 @@
 		    <material name="white"/>
 		</collision>
+        <inertial>
+			<mass value="${caster_mass}"/>
+			<xacro:sphere_inertia mass="${caster_mass}" r="0.0095" />
+		</inertial>
 	</link>
     <!-- Implement the left wheel -->
@@ -107,4 +112,5 @@
 		<origin xyz="-0.03 0.056 -0.0100" rpy="0 0 0"/>
 		<axis xyz="0 1 0"/>
+        <dynamics friction="${left_wheel_mu_p}"/>
 	</joint>
     <!-- Implement the joint for the right wheel -->
@@ -114,4 +120,5 @@
 		<origin xyz="-0.03 -0.056 -0.0100" rpy="0 0 0"/>
 		<axis xyz="0 1 0"/>
+        <dynamics friction="${right_wheel_mu_p}"/>
 	</joint>
     <!-- Add your sensors using the macro -->

Commit message: update urdf and python

File: ros_basics_exercise/urdf/thymio_simple.urdf.xacro (robot description, xacro)
@@ -13,7 +13,7 @@
     <xacro:arg name="mass" default="0.270"/>
     <xacro:property name="mass_p" value="$(arg mass)"/>
-    <xacro:property name="body_mass" value="${mass_p * 0.75}"/>
+    <xacro:property name="body_mass" value="${mass_p * 0.78}"/>
     <xacro:property name="wheel_mass" value="${mass_p * 0.10}"/>
-    <xacro:property name="caster_mass" value="${mass_p * 0.05}"/>
+    <xacro:property name="caster_mass" value="${mass_p * 0.02}"/>
     <link name="base_link">
         <visual>

Commit message: session 2

File: ros_basics_exercise/urdf/thymio_simple.urdf.xacro (robot description, xacro)
@@ -103,5 +103,5 @@
 		<parent link="base_link"/>
 		<child link="caster_wheel"/>
-		<origin xyz="0.03 0 -0.0225" rpy="0 0 0"/>
+		<origin xyz="0.045 0 -0.0225" rpy="0 0 0"/>
 		<axis xyz="0 0 0"/>
 	</joint>
@@ -110,5 +110,5 @@
 		<parent link="base_link"/>
 		<child link="left_wheel"/>
-		<origin xyz="-0.03 0.056 -0.0100" rpy="0 0 0"/>
+		<origin xyz="-0.02 0.056 -0.0100" rpy="0 0 0"/>
 		<axis xyz="0 1 0"/>
         <dynamics friction="${left_wheel_mu_p}"/>
@@ -118,8 +118,15 @@
 		<parent link="base_link"/>
 		<child link="right_wheel"/>
-		<origin xyz="-0.03 -0.056 -0.0100" rpy="0 0 0"/>
+		<origin xyz="-0.02 -0.056 -0.0100" rpy="0 0 0"/>
 		<axis xyz="0 1 0"/>
         <dynamics friction="${right_wheel_mu_p}"/>
 	</joint>
     <!-- Add your sensors using the macro -->
+    <xacro:csensor plink="base_link" id="0" mass="0.001" originrpy="0 0 0" originxyz="-0.003 0 0" jointxyz="0.0600 0.0450 0" jointrpy="${pi} 0 ${pi/2 + pi/6}"/>
+    <xacro:csensor plink="base_link" id="1" mass="0.001" originrpy="0 0 0" originxyz="-0.003 0 0" jointxyz="0.0650 0.0225 0" jointrpy="${pi} 0 ${pi/2 + pi/12}"/>
+    <xacro:csensor plink="base_link" id="2" mass="0.001" originrpy="0 0 0" originxyz="-0.003 0 0" jointxyz="0.0700 0 0" jointrpy="${pi} 0 ${pi/2}"/>
+    <xacro:csensor plink="base_link" id="3" mass="0.001" originrpy="0 0 0" originxyz="-0.003 0 0" jointxyz="0.0600 -0.0450 0" jointrpy="0 0 -${pi/2 + pi/6}"/>
+    <xacro:csensor plink="base_link" id="4" mass="0.001" originrpy="0 0 0" originxyz="-0.003 0 0" jointxyz="0.0650 -0.0225 0" jointrpy="0 0 -${pi/2 + pi/12}"/>
+    <xacro:csensor plink="base_link" id="5" mass="0.001" originrpy="0 0 0" originxyz="-0.003 0 0" jointxyz="-0.056 -0.03 0" jointrpy="0 0 ${pi/2}"/>
+    <xacro:csensor plink="base_link" id="6" mass="0.001" originrpy="0 0 0" originxyz="-0.003 0 0" jointxyz="-0.056 0.03 0" jointrpy="0 0 ${pi/2}"/>
 </robot>

Commit message: plot in coming

File: ros_basics_exercise/urdf/thymio_simple.urdf.xacro (robot description, xacro)
@@ -99,4 +99,24 @@
 		</inertial>
     </link>
+    <link name="obs">
+        <visual>
+            <origin xyz="0 0 0" rpy="0 0 0"/>
+            <geometry>
+                <box size="0.033 0.065 0.07"/>
+            </geometry>
+            <material name="white"/>
+        </visual>
+        <collision>
+            <origin xyz="0 0 0" rpy="0 0 0"/>
+            <geometry>
+                <box size="0.033 0.065 0.07"/>
+            </geometry>
+            <material name="white"/>
+        </collision>
+        <inertial>
+			<mass value="0.100"/>
+			<xacro:box_inertia mass="0.100" x="0.11" y="0.112" z="0.045" />
+		</inertial>
+    </link>
     <!-- Implement the joint for the caster wheel -->
 	<joint name="caster_wheel_joint" type="fixed">

Commit message: simu done

File: ros_basics_exercise/urdf/thymio_simple.urdf.xacro (robot description, xacro)
@@ -99,24 +99,4 @@
 		</inertial>
     </link>
-    <link name="obs">
-        <visual>
-            <origin xyz="0 0 0" rpy="0 0 0"/>
-            <geometry>
-                <box size="0.033 0.065 0.07"/>
-            </geometry>
-            <material name="white"/>
-        </visual>
-        <collision>
-            <origin xyz="0 0 0" rpy="0 0 0"/>
-            <geometry>
-                <box size="0.033 0.065 0.07"/>
-            </geometry>
-            <material name="white"/>
-        </collision>
-        <inertial>
-			<mass value="0.100"/>
-			<xacro:box_inertia mass="0.100" x="0.11" y="0.112" z="0.045" />
-		</inertial>
-    </link>
     <!-- Implement the joint for the caster wheel -->
 	<joint name="caster_wheel_joint" type="fixed">
@@ -130,5 +110,5 @@
 		<parent link="base_link"/>
 		<child link="left_wheel"/>
-		<origin xyz="-0.02 0.056 -0.0100" rpy="0 0 0"/>
+		<origin xyz="-0.02 0.0485 -0.0100" rpy="0 0 0"/>
 		<axis xyz="0 1 0"/>
         <dynamics friction="${left_wheel_mu_p}"/>
@@ -138,14 +118,14 @@
 		<parent link="base_link"/>
 		<child link="right_wheel"/>
-		<origin xyz="-0.02 -0.056 -0.0100" rpy="0 0 0"/>
+		<origin xyz="-0.02 -0.0485 -0.0100" rpy="0 0 0"/>
 		<axis xyz="0 1 0"/>
         <dynamics friction="${right_wheel_mu_p}"/>
 	</joint>
     <!-- Add your sensors using the macro -->
-    <xacro:csensor plink="base_link" id="0" mass="0.001" originrpy="0 0 0" originxyz="-0.003 0 0" jointxyz="0.0600 0.0450 0" jointrpy="${pi} 0 ${pi/2 + pi/6}"/>
-    <xacro:csensor plink="base_link" id="1" mass="0.001" originrpy="0 0 0" originxyz="-0.003 0 0" jointxyz="0.0650 0.0225 0" jointrpy="${pi} 0 ${pi/2 + pi/12}"/>
+    <xacro:csensor plink="base_link" id="0" mass="0.001" originrpy="0 0 0" originxyz="-0.003 0 0" jointxyz="0.0600 0.0575 0" jointrpy="${pi} 0 ${pi/2 + pi/6}"/>
+    <xacro:csensor plink="base_link" id="1" mass="0.001" originrpy="0 0 0" originxyz="-0.003 0 0" jointxyz="0.0650 0.0325 0" jointrpy="${pi} 0 ${pi/2 + pi/12}"/>
     <xacro:csensor plink="base_link" id="2" mass="0.001" originrpy="0 0 0" originxyz="-0.003 0 0" jointxyz="0.0700 0 0" jointrpy="${pi} 0 ${pi/2}"/>
-    <xacro:csensor plink="base_link" id="3" mass="0.001" originrpy="0 0 0" originxyz="-0.003 0 0" jointxyz="0.0600 -0.0450 0" jointrpy="0 0 -${pi/2 + pi/6}"/>
-    <xacro:csensor plink="base_link" id="4" mass="0.001" originrpy="0 0 0" originxyz="-0.003 0 0" jointxyz="0.0650 -0.0225 0" jointrpy="0 0 -${pi/2 + pi/12}"/>
+    <xacro:csensor plink="base_link" id="3" mass="0.001" originrpy="0 0 0" originxyz="-0.003 0 0" jointxyz="0.0650 -0.0325 0" jointrpy="0 0 -${pi/2 + pi/12}"/>
+    <xacro:csensor plink="base_link" id="4" mass="0.001" originrpy="0 0 0" originxyz="-0.003 0 0" jointxyz="0.0600 -0.0575 0" jointrpy="0 0 -${pi/2 + pi/6}"/>
     <xacro:csensor plink="base_link" id="5" mass="0.001" originrpy="0 0 0" originxyz="-0.003 0 0" jointxyz="-0.056 -0.03 0" jointrpy="0 0 ${pi/2}"/>
     <xacro:csensor plink="base_link" id="6" mass="0.001" originrpy="0 0 0" originxyz="-0.003 0 0" jointxyz="-0.056 0.03 0" jointrpy="0 0 ${pi/2}"/>
